File: hardware/V0.0.3/lambda_bl49.sch (EAGLE design)
At the start: 58 parts, among them IC10 MCP2551-E/SN, IC3 LMV321IDBVR, IC4 TLS115B0EJXUMA1, IC6 TLE4270-2D, IC9 CJ125_32, Q3 ABM3-16.000MHZ-D2Y-T

Commit message: tls115 replaced by ti ref5050
Parts:
- removed IC4: TLS115B0EJXUMA1, Heinrich:TLS115B0EJXUMA1
- added D2: P6SMB18A, Heinrich:P6SMBXXASMB
- added IC1: REF50XX, Heinrich:REF50XX
- D1: value SMBJ36CA -> S1J; device Heinrich:P6SMBXXCA -> Heinrich:DIODESMA
Connections:
- new net VBAT: C1.1, C14.1, C15.+, C6.+, D1.C, D2.C, IC1.VIN, IC6.I
- net +5V: no longer IC4.ADJ
- net +UB: now also D1.A; no longer C1.1, C14.1, C15.+, C6.+, D1.2, IC4.EN, IC4.IN, IC6.I
- net AREF: now also IC1.VOUT; no longer IC4.OUT
- net GND: now also D2.A, IC1.GND; no longer D1.1, IC4.GND
